Commit message: added ros2_control

File: description/robot1.urdf.xacro (robot description, xacro)
@@ -2,3 +2,5 @@
 <robot xmlns:xacro="http://www.ros.org/wiki/xacro" name="my_robot1">
     <xacro:include filename="robot1_core.xacro"/>
+    <xacro:include filename="ros2_control.xacro"/>
+    <!-- <xacro:include filename="gazebo_control.xacro"/> -->
 </robot>

File: description/robot1_core.xacro (robot description, xacro)
@@ -39,4 +39,7 @@
         </xacro:inertial_box>
     </link>
+    <gazebo reference="chassis">
+        <material>Gazebo/White</material>
+    </gazebo>
     <joint name="base_to_box_joint" type="fixed">
         <parent link="base_link"/>
@@ -63,4 +66,7 @@
         </xacro:inertial_cylinder>
     </link>
+    <gazebo reference="wheel_axis_link">
+        <material>Gazebo/Green</material>
+    </gazebo>
     <joint name="base_to_wheel_axis" type="fixed">
         <parent link="base_link"/>
@@ -87,4 +93,7 @@
         </xacro:inertial_cylinder>
     </link>
+    <gazebo reference="left_wheel">
+        <material>Gazebo/Blue</material>
+    </gazebo>
     <joint name="base_to_left_wheel" type="continuous">
         <parent link="base_link"/>
@@ -112,4 +121,7 @@
         </xacro:inertial_cylinder>
     </link>
+    <gazebo reference="right_wheel">
+        <material>Gazebo/Blue</material>
+    </gazebo>
     <joint name="base_to_right_wheel" type="continuous">
         <parent link="base_link"/>
@@ -137,4 +149,9 @@
         </xacro:inertial_sphere>
     </link>
+    <gazebo reference="rear_pivot">
+        <material>Gazebo/Blue</material>
+        <mu1 value="0.001"/>
+        <mu2 value="0.001"/>
+    </gazebo>
     <joint name="base_to_rear_pivot" type="fixed">
         <parent link="base_link"/>
